File: hardware/cm4-carrier-template/cm4-carrier-template.sch (KiCad schematic (older format))
At the start: 26 parts, among them J1 USB_C_Receptacle_USB2.0, J2 Micro_SD_Card, J3 Abracon_ARJ-139, U1 TPD2EUSB30, U2 TPD2EUSB30, U3 TPD2EUSB30, U4 TPD2EUSB30, U5 Compute_Module_4_Functional, U6 Expansion_PoE

Commit message: Pre-stream commit.
Parts:
- removed J3: Abracon_ARJ-139, jkiv-library:RJ45_Abracon_ARJ136, symbol jkiv-abracon:Abracon_ARJ-139
- removed JP1: USB_VBUS, Jumper:SolderJumper-2_P1.3mm_Bridged_RoundedPad1.0x1.5mm, symbol Device:Jumper_NC_Small
- removed JP2: USB_GND, Jumper:SolderJumper-2_P1.3mm_Bridged_RoundedPad1.0x1.5mm, symbol Device:Jumper_NC_Small
- removed L1: DNP, Inductor_SMD:L_CommonMode_Wuerth_WE-SL2, symbol Device:L_Core_Ferrite_Coupled_1423
- removed U1, U2, U3, U4: TPD2EUSB30, Package_TO_SOT_SMD:Texas_DRT-3, symbol Power_Protection:TPD2EUSB30
- removed U6: Expansion_PoE, jkiv-library:expansion-poe-P2.0mm_SMD, symbol jkiv-expansion:Expansion_PoE
- added C2: 22u, Capacitor_SMD:C_0805_2012Metric, symbol Device:C_Small
- added C3: 100n, Capacitor_SMD:C_0805_2012Metric, symbol Device:C_Small
- added D2: RPi 3v3, LED_SMD:LED_0603_1608Metric, symbol Device:LED_Small
- added D3: Activity LED, LED_SMD:LED_0603_1608Metric, symbol Device:LED_Small
- added D4: SD ON, LED_SMD:LED_0603_1608Metric, symbol Device:LED_Small
- added FB1: FB, Inductor_SMD:L_0805_2012Metric, symbol Device:Ferrite_Bead_Small
- added FID4, FID5, FID6: Fiducial, Fiducial:Fiducial_0.75mm_Mask1.5mm, symbol Mechanical:Fiducial
- added J3: Abracon_ARJM11-502, jkiv-library:RJ45_Abracon_ARJM11, symbol jkiv-abracon:Abracon_ARJM11-502
- added Q1: DMP2066LSN, Package_TO_SOT_SMD:SC-59, symbol Device:Q_PMOS_GSD
- added R10, R11, R12, R7, R8, R9: 220R, Resistor_SMD:R_0603_1608Metric, symbol Device:R_Small_US
- added R13, R14, R15: 0R, Resistor_SMD:R_0603_1608Metric, symbol Device:R_Small_US
- added R6: 330R, Resistor_SMD:R_0603_1608Metric, symbol Device:R_Small_US
- added SW1: BOOT, Button_Switch_SMD:SW_SPST_B3U-1000P, symbol Switch:SW_Push
- added SW2: GLOBAL_EN, Button_Switch_SMD:SW_SPST_B3U-1000P, symbol Switch:SW_Push
- added U6: TPD2EUSB30, Package_TO_SOT_SMD:Texas_DRT-3, symbol Power_Protection:TPD2EUSB30
- D1: value SD ON -> USB Power; footprint Diode_SMD:D_0603_1608Metric -> LED_SMD:LED_0603_1608Metric
- R3, R4: value 100R -> 220R
- R5: value 100R -> DNP
Connections:
- net labels added: PI_GLOBAL_EN, PI_LED_nACT, PI_nRPI_BOOT, SD_PWR, SD_PWR_ON
- net labels removed: E0_TD0+, E0_TD0-, E0_TD1+, E0_TD1-, E0_TD2+, E0_TD2-, E0_TD3+, E0_TD3-, GNDREF, PoE_TAP1, PoE_TAP2, PoE_TAP3, PoE_TAP4, USB_GND, VBUS
- wire segments 119 -> 131
- no-connect marks 49 -> 48
Other:
- note added: "Gigabit Ethernet"
- note added: "Hold to boot from USB"
- note added: "Low for <1ms to Power Up"
- note added: "Remove shorts to enable features."
- note added: "Short if eMMC (1.8V)"
- note added: "USB Type-C Power (5V@3A)\nUSB 2.0 Data"
- note removed: "Gigabit Ethernet with PoE+"
- note removed: "TODO"
- note removed: "TODO CT"
- note removed: "TODO host"
- note removed: "USB Type-C Power (5V@3A)"
- moved on the sheet: C1, FID1, FID2, FID3, J1, R1, R2, R3, R4, U5C
